Commit message: test

File: hexapod_description/urdf/hexaforce_visuals_collisions.xacro (robot description, xacro)
@@ -51,9 +51,9 @@
   <xacro:macro name="visuals_collisions_leg_1">
     <visual>
-      <origin xyz="0 0 0" rpy="0 ${PI_2} 0"/>
+      <origin xyz="0 0.75 0" rpy="-${PI} 0 0"/>
         <geometry>
           <mesh filename="${path_prefix + 'stl/first_link.stl'}" scale="0.001 0.001 0.001"/>
         </geometry>
-      <material name="Red"/>
+      <material name="Green"/>
     </visual>
     <collision>
@@ -66,5 +66,5 @@
   <xacro:macro name="visuals_collisions_leg_2">
     <visual>
-      <origin xyz="0 0 0" rpy="0 -${PI_2} 0"/>
+      <origin xyz="0 0 0" rpy="${PI_2} ${PI} ${PI_2}"/>
         <geometry>
           <mesh filename="${path_prefix + 'stl/second_link.stl'}" scale="0.001 0.001 0.001"/>

File: hexapod_description/urdf/modules/leg_hexaforce.xacro (robot description, xacro)
@@ -2,5 +2,5 @@
 <robot xmlns:xacro="http://www.ros.org/wiki/xacro">
     <!-- XACRO MACRO FOR LEGS LINKS/JOINTS -->
-    <xacro:macro name="leg" params="index xPos yPos">
+    <xacro:macro name="leg" params="index xPos yPos zPos">
         <joint name="body_leg_${index}" type="revolute">
             <parent link="base_link"/>
@@ -22,5 +22,5 @@
                 <xacro:property name="legs_rotation" value="${PI}"/>
             </xacro:if>
-            <origin rpy="0 0 ${offset_angle+legs_rotation}" xyz="${xPos} ${yPos} 0"/>
+            <origin rpy="0 0 ${offset_angle+legs_rotation}" xyz="${xPos} ${yPos} ${zPos}"/>
             <axis xyz="0 0 1"/>
             <dynamics damping="${joint_dmp}" friction="${joint_friction}"/>
@@ -40,5 +40,5 @@
             <child link="leg_${index}_2"/>
             <limit effort="${joint_eff}" lower="${-joint_lim}" upper="${joint_lim}" velocity="${joint_vel}"/>
-            <origin rpy="0 0 0" xyz="0 ${leg1_length} 0"/>
+            <origin rpy="0 0 0" xyz="-0.2 ${leg1_length+0.7} -0.2"/>
             <axis xyz="1 0 0"/>
             <dynamics damping="${joint_dmp}" friction="${joint_friction}"/>
@@ -58,5 +58,5 @@
             <child link="leg_${index}_3"/>
             <limit effort="${joint_eff}" lower="${-joint_lim}" upper="${joint_lim}" velocity="${joint_vel}"/>
-            <origin rpy="0 0 0" xyz="0 ${leg2_length} 0"/>
+            <origin rpy="0 0 0" xyz="0.2 ${leg2_length+1} 0"/>
             <axis xyz="-1 0 0"/>
             <dynamics damping="${joint_dmp}" friction="${joint_friction}"/>

File: hexapod_description/urdf/modules/legs_hexaforce.xacro (robot description, xacro)
@@ -2,10 +2,10 @@
 <robot xmlns:xacro="http://www.ros.org/wiki/xacro">
   <!-- LEGS LINKS/JOINTS -->
-    <xacro:leg index="2" xPos="${body_length/2}" yPos="${body_width/2}"/>
-    <xacro:leg index="3" xPos="${body_length/2}" yPos="${-body_width/2}"/>
-    <xacro:leg index="0" xPos="${-body_length/2}" yPos="${body_width/2}"/>
-    <xacro:leg index="5" xPos="${-body_length/2}" yPos="${-body_width/2}"/>
-    <xacro:leg index="1" xPos="0" yPos="${body_width_extra/2}"/>
-    <xacro:leg index="4" xPos="0" yPos="${-body_width_extra/2}"/>
+    <xacro:leg index="2" xPos="${body_length/2+1.2}" yPos="${body_width/2+0.8}" zPos="1.2"/>
+    <xacro:leg index="3" xPos="${body_length/2+1.2}" yPos="${-body_width/2-0.8}" zPos="1.2"/>
+    <xacro:leg index="0" xPos="${-body_length/2-1.1}" yPos="${body_width/2+0.8}" zPos="1.2"/>
+    <xacro:leg index="5" xPos="${-body_length/2-1.1}" yPos="${-body_width/2-0.8}" zPos="1.2"/>
+    <xacro:leg index="1" xPos="0" yPos="${body_width_extra/2+0.8}" zPos="1.2"/>
+    <xacro:leg index="4" xPos="0" yPos="${-body_width_extra/2-0.8}" zPos="1.2"/>
   <!-- END OF LEG LINKS/JOINTS -->
 </robot>
