Commit message: also edited pexod.urdf

File: hexapod_description/hexaforce.urdf (robot description, URDF)
Before this commit: robot pexod, 25 links, 24 joints
Links:
- link base_link: mass 1.031 -> 1.834
- link leg_0_1: mass 0.02 -> 0.073
- link leg_0_2: mass 0.184 -> 0.02
- link leg_0_3: mass 0.04 -> 0.08
- link leg_1_1: mass 0.02 -> 0.073
- link leg_1_2: mass 0.184 -> 0.02
- link leg_1_3: mass 0.04 -> 0.08
- link leg_2_1: mass 0.02 -> 0.073
- link leg_2_2: mass 0.184 -> 0.02
- link leg_2_3: mass 0.04 -> 0.08
- link leg_3_1: mass 0.02 -> 0.073
- link leg_3_2: mass 0.184 -> 0.02
- link leg_3_3: mass 0.04 -> 0.08
- link leg_4_1: mass 0.02 -> 0.073
- link leg_4_2: mass 0.184 -> 0.02
- link leg_4_3: mass 0.04 -> 0.08
- link leg_5_1: mass 0.02 -> 0.073
- link leg_5_2: mass 0.184 -> 0.02
- link leg_5_3: mass 0.04 -> 0.08
Joints:
- joint leg_0_2_3: limit lower=-1.57079632679 upper=1.57079632679 effort=2.5 velocity=5.75958653158 -> lower=-1.57079632679 upper=0.82 effort=2.5 velocity=5.75958653158
- joint leg_1_2_3: limit lower=-1.57079632679 upper=1.57079632679 effort=2.5 velocity=5.75958653158 -> lower=-1.57079632679 upper=0.82 effort=2.5 velocity=5.75958653158
- joint leg_2_2_3: limit lower=-1.57079632679 upper=1.57079632679 effort=2.5 velocity=5.75958653158 -> lower=-1.57079632679 upper=0.82 effort=2.5 velocity=5.75958653158
- joint leg_3_2_3: limit lower=-1.57079632679 upper=1.57079632679 effort=2.5 velocity=5.75958653158 -> lower=-1.57079632679 upper=0.82 effort=2.5 velocity=5.75958653158
- joint leg_4_2_3: limit lower=-1.57079632679 upper=1.57079632679 effort=2.5 velocity=5.75958653158 -> lower=-1.57079632679 upper=0.82 effort=2.5 velocity=5.75958653158
- joint leg_5_2_3: limit lower=-1.57079632679 upper=1.57079632679 effort=2.5 velocity=5.75958653158 -> lower=-1.57079632679 upper=0.82 effort=2.5 velocity=5.75958653158

File: hexapod_description/hexaforce_simulation.urdf (robot description, URDF)
Before this commit: robot pexod, 25 links, 24 joints
Links:
- link base_link: mass 1.031 -> 1.834
- link leg_0_1: mass 0.02 -> 0.073
- link leg_0_2: mass 0.184 -> 0.02
- link leg_0_3: mass 0.04 -> 0.08
- link leg_1_1: mass 0.02 -> 0.073
- link leg_1_2: mass 0.184 -> 0.02
- link leg_1_3: mass 0.04 -> 0.08
- link leg_2_1: mass 0.02 -> 0.073
- link leg_2_2: mass 0.184 -> 0.02
- link leg_2_3: mass 0.04 -> 0.08
- link leg_3_1: mass 0.02 -> 0.073
- link leg_3_2: mass 0.184 -> 0.02
- link leg_3_3: mass 0.04 -> 0.08
- link leg_4_1: mass 0.02 -> 0.073
- link leg_4_2: mass 0.184 -> 0.02
- link leg_4_3: mass 0.04 -> 0.08
- link leg_5_1: mass 0.02 -> 0.073
- link leg_5_2: mass 0.184 -> 0.02
- link leg_5_3: mass 0.04 -> 0.08
Joints:
- joint leg_0_2_3: limit lower=-1.57079632679 upper=1.57079632679 effort=2.5 velocity=5.75958653158 -> lower=-1.57079632679 upper=0.82 effort=2.5 velocity=5.75958653158
- joint leg_1_2_3: limit lower=-1.57079632679 upper=1.57079632679 effort=2.5 velocity=5.75958653158 -> lower=-1.57079632679 upper=0.82 effort=2.5 velocity=5.75958653158
- joint leg_2_2_3: limit lower=-1.57079632679 upper=1.57079632679 effort=2.5 velocity=5.75958653158 -> lower=-1.57079632679 upper=0.82 effort=2.5 velocity=5.75958653158
- joint leg_3_2_3: limit lower=-1.57079632679 upper=1.57079632679 effort=2.5 velocity=5.75958653158 -> lower=-1.57079632679 upper=0.82 effort=2.5 velocity=5.75958653158
- joint leg_4_2_3: limit lower=-1.57079632679 upper=1.57079632679 effort=2.5 velocity=5.75958653158 -> lower=-1.57079632679 upper=0.82 effort=2.5 velocity=5.75958653158
- joint leg_5_2_3: limit lower=-1.57079632679 upper=1.57079632679 effort=2.5 velocity=5.75958653158 -> lower=-1.57079632679 upper=0.82 effort=2.5 velocity=5.75958653158

File: hexapod_description/pexod.urdf (robot description, URDF)
Before this commit: robot pexod, 19 links, 18 joints
Links:
- link base_link: mass 1.031 -> 1.834
- link leg_0_1: mass 0.02 -> 0.073
- link leg_0_2: mass 0.184 -> 0.02
- link leg_0_3: mass 0.04 -> 0.08
- link leg_1_1: mass 0.02 -> 0.073
- link leg_1_2: mass 0.184 -> 0.02
- link leg_1_3: mass 0.04 -> 0.08
- link leg_2_1: mass 0.02 -> 0.073
- link leg_2_2: mass 0.184 -> 0.02
- link leg_2_3: mass 0.04 -> 0.08
- link leg_3_1: mass 0.02 -> 0.073
- link leg_3_2: mass 0.184 -> 0.02
- link leg_3_3: mass 0.04 -> 0.08
- link leg_4_1: mass 0.02 -> 0.073
- link leg_4_2: mass 0.184 -> 0.02
- link leg_4_3: mass 0.04 -> 0.08
- link leg_5_1: mass 0.02 -> 0.073
- link leg_5_2: mass 0.184 -> 0.02
- link leg_5_3: mass 0.04 -> 0.08
Joints:
- joint body_leg_0: origin xyz=-0.12 0.0595 0 rpy=0 0 0.3 -> xyz=-1.22 0.8595 1.2 rpy=0 0 0.3
- joint body_leg_1: origin xyz=0 0.0995 0 rpy=0 0 0 -> xyz=0 0.8995 1.2 rpy=0 0 0
- joint body_leg_2: origin xyz=0.12 0.0595 0 rpy=0 0 -0.3 -> xyz=1.32 0.8595 1.2 rpy=0 0 -0.3
- joint body_leg_3: origin xyz=0.12 -0.0595 0 rpy=0 0 3.44159265359 -> xyz=1.32 -0.8595 1.2 rpy=0 0 3.44159265359
- joint body_leg_4: origin xyz=0 -0.0995 0 rpy=0 0 3.14159265359 -> xyz=0 -0.8995 1.2 rpy=0 0 3.14159265359
- joint body_leg_5: origin xyz=-0.12 -0.0595 0 rpy=0 0 2.84159265359 -> xyz=-1.22 -0.8595 1.2 rpy=0 0 2.84159265359
- joint leg_0_1_2: origin xyz=0 0.06 0 rpy=0 0 0 -> xyz=-0.2 0.76 -0.2 rpy=0 0 0
- joint leg_0_2_3: limit lower=-1.57079632679 upper=1.57079632679 effort=2.5 velocity=5.75958653158 -> lower=-1.57079632679 upper=0.82 effort=2.5 velocity=5.75958653158; origin xyz=0 0.0835 0 rpy=0 0 0 -> xyz=0.2 1.0835 0 rpy=0 0 0
- joint leg_1_1_2: origin xyz=0 0.06 0 rpy=0 0 0 -> xyz=-0.2 0.76 -0.2 rpy=0 0 0
- joint leg_1_2_3: limit lower=-1.57079632679 upper=1.57079632679 effort=2.5 velocity=5.75958653158 -> lower=-1.57079632679 upper=0.82 effort=2.5 velocity=5.75958653158; origin xyz=0 0.0835 0 rpy=0 0 0 -> xyz=0.2 1.0835 0 rpy=0 0 0
- joint leg_2_1_2: origin xyz=0 0.06 0 rpy=0 0 0 -> xyz=-0.2 0.76 -0.2 rpy=0 0 0
- joint leg_2_2_3: limit lower=-1.57079632679 upper=1.57079632679 effort=2.5 velocity=5.75958653158 -> lower=-1.57079632679 upper=0.82 effort=2.5 velocity=5.75958653158; origin xyz=0 0.0835 0 rpy=0 0 0 -> xyz=0.2 1.0835 0 rpy=0 0 0
- joint leg_3_1_2: origin xyz=0 0.06 0 rpy=0 0 0 -> xyz=-0.2 0.76 -0.2 rpy=0 0 0
- joint leg_3_2_3: limit lower=-1.57079632679 upper=1.57079632679 effort=2.5 velocity=5.75958653158 -> lower=-1.57079632679 upper=0.82 effort=2.5 velocity=5.75958653158; origin xyz=0 0.0835 0 rpy=0 0 0 -> xyz=0.2 1.0835 0 rpy=0 0 0
- joint leg_4_1_2: origin xyz=0 0.06 0 rpy=0 0 0 -> xyz=-0.2 0.76 -0.2 rpy=0 0 0
- joint leg_4_2_3: limit lower=-1.57079632679 upper=1.57079632679 effort=2.5 velocity=5.75958653158 -> lower=-1.57079632679 upper=0.82 effort=2.5 velocity=5.75958653158; origin xyz=0 0.0835 0 rpy=0 0 0 -> xyz=0.2 1.0835 0 rpy=0 0 0
- joint leg_5_1_2: origin xyz=0 0.06 0 rpy=0 0 0 -> xyz=-0.2 0.76 -0.2 rpy=0 0 0
- joint leg_5_2_3: limit lower=-1.57079632679 upper=1.57079632679 effort=2.5 velocity=5.75958653158 -> lower=-1.57079632679 upper=0.82 effort=2.5 velocity=5.75958653158; origin xyz=0 0.0835 0 rpy=0 0 0 -> xyz=0.2 1.0835 0 rpy=0 0 0

File: hexapod_description/pexod_simulation.urdf (robot description, URDF)
Before this commit: robot pexod, 19 links, 18 joints
Links:
- link base_link: mass 1.031 -> 1.834
- link leg_0_1: mass 0.02 -> 0.073
- link leg_0_2: mass 0.184 -> 0.02
- link leg_0_3: mass 0.04 -> 0.08
- link leg_1_1: mass 0.02 -> 0.073
- link leg_1_2: mass 0.184 -> 0.02
- link leg_1_3: mass 0.04 -> 0.08
- link leg_2_1: mass 0.02 -> 0.073
- link leg_2_2: mass 0.184 -> 0.02
- link leg_2_3: mass 0.04 -> 0.08
- link leg_3_1: mass 0.02 -> 0.073
- link leg_3_2: mass 0.184 -> 0.02
- link leg_3_3: mass 0.04 -> 0.08
- link leg_4_1: mass 0.02 -> 0.073
- link leg_4_2: mass 0.184 -> 0.02
- link leg_4_3: mass 0.04 -> 0.08
- link leg_5_1: mass 0.02 -> 0.073
- link leg_5_2: mass 0.184 -> 0.02
- link leg_5_3: mass 0.04 -> 0.08
Joints:
- joint body_leg_0: origin xyz=-0.12 0.0595 0 rpy=0 0 0.3 -> xyz=-1.22 0.8595 1.2 rpy=0 0 0.3
- joint body_leg_1: origin xyz=0 0.0995 0 rpy=0 0 0 -> xyz=0 0.8995 1.2 rpy=0 0 0
- joint body_leg_2: origin xyz=0.12 0.0595 0 rpy=0 0 -0.3 -> xyz=1.32 0.8595 1.2 rpy=0 0 -0.3
- joint body_leg_3: origin xyz=0.12 -0.0595 0 rpy=0 0 3.44159265359 -> xyz=1.32 -0.8595 1.2 rpy=0 0 3.44159265359
- joint body_leg_4: origin xyz=0 -0.0995 0 rpy=0 0 3.14159265359 -> xyz=0 -0.8995 1.2 rpy=0 0 3.14159265359
- joint body_leg_5: origin xyz=-0.12 -0.0595 0 rpy=0 0 2.84159265359 -> xyz=-1.22 -0.8595 1.2 rpy=0 0 2.84159265359
- joint leg_0_1_2: origin xyz=0 0.06 0 rpy=0 0 0 -> xyz=-0.2 0.76 -0.2 rpy=0 0 0
- joint leg_0_2_3: limit lower=-1.57079632679 upper=1.57079632679 effort=2.5 velocity=5.75958653158 -> lower=-1.57079632679 upper=0.82 effort=2.5 velocity=5.75958653158; origin xyz=0 0.0835 0 rpy=0 0 0 -> xyz=0.2 1.0835 0 rpy=0 0 0
- joint leg_1_1_2: origin xyz=0 0.06 0 rpy=0 0 0 -> xyz=-0.2 0.76 -0.2 rpy=0 0 0
- joint leg_1_2_3: limit lower=-1.57079632679 upper=1.57079632679 effort=2.5 velocity=5.75958653158 -> lower=-1.57079632679 upper=0.82 effort=2.5 velocity=5.75958653158; origin xyz=0 0.0835 0 rpy=0 0 0 -> xyz=0.2 1.0835 0 rpy=0 0 0
- joint leg_2_1_2: origin xyz=0 0.06 0 rpy=0 0 0 -> xyz=-0.2 0.76 -0.2 rpy=0 0 0
- joint leg_2_2_3: limit lower=-1.57079632679 upper=1.57079632679 effort=2.5 velocity=5.75958653158 -> lower=-1.57079632679 upper=0.82 effort=2.5 velocity=5.75958653158; origin xyz=0 0.0835 0 rpy=0 0 0 -> xyz=0.2 1.0835 0 rpy=0 0 0
- joint leg_3_1_2: origin xyz=0 0.06 0 rpy=0 0 0 -> xyz=-0.2 0.76 -0.2 rpy=0 0 0
- joint leg_3_2_3: limit lower=-1.57079632679 upper=1.57079632679 effort=2.5 velocity=5.75958653158 -> lower=-1.57079632679 upper=0.82 effort=2.5 velocity=5.75958653158; origin xyz=0 0.0835 0 rpy=0 0 0 -> xyz=0.2 1.0835 0 rpy=0 0 0
- joint leg_4_1_2: origin xyz=0 0.06 0 rpy=0 0 0 -> xyz=-0.2 0.76 -0.2 rpy=0 0 0
- joint leg_4_2_3: limit lower=-1.57079632679 upper=1.57079632679 effort=2.5 velocity=5.75958653158 -> lower=-1.57079632679 upper=0.82 effort=2.5 velocity=5.75958653158; origin xyz=0 0.0835 0 rpy=0 0 0 -> xyz=0.2 1.0835 0 rpy=0 0 0
- joint leg_5_1_2: origin xyz=0 0.06 0 rpy=0 0 0 -> xyz=-0.2 0.76 -0.2 rpy=0 0 0
- joint leg_5_2_3: limit lower=-1.57079632679 upper=1.57079632679 effort=2.5 velocity=5.75958653158 -> lower=-1.57079632679 upper=0.82 effort=2.5 velocity=5.75958653158; origin xyz=0 0.0835 0 rpy=0 0 0 -> xyz=0.2 1.0835 0 rpy=0 0 0

File: hexapod_description/urdf/modules/hexaforce.xacro (robot description, xacro)
@@ -6,5 +6,5 @@
   <xacro:property name="PI_4" value="0.78539816339" />
   <xacro:property name="scale" value="0.001" />
-  <xacro:property name="body_mass" value="1.031"/>
+  <xacro:property name="body_mass" value="1.834"/>
   <xacro:property name="body_length" value="0.24"/>
   <xacro:property name="body_width" value="0.119"/>
@@ -14,14 +14,14 @@
   <xacro:property name="leg1_length" value="0.06"/>
   <xacro:property name="leg1_dist" value="0.2"/>
-  <xacro:property name="leg1_mass" value="0.02"/>
+  <xacro:property name="leg1_mass" value="0.073"/>
   <xacro:property name="leg2_width" value="0.038"/>
   <xacro:property name="leg2_length" value="0.0835"/>
   <xacro:property name="leg2_dist" value="0.2"/>
-  <xacro:property name="leg2_mass" value="0.184"/>
+  <xacro:property name="leg2_mass" value="0.02"/>
   <xacro:property name="leg3_width" value="0.054"/>
   <xacro:property name="leg3_length" value="0.065"/>
   <xacro:property name="leg3_height" value="0.10"/>
   <xacro:property name="leg3_tip_radius" value="0.02"/>
-  <xacro:property name="leg3_mass" value="0.04"/>
+  <xacro:property name="leg3_mass" value="0.08"/>
   <xacro:property name="force_y_offset" value="${(11.25+27)*0.001}"/>
   <xacro:property name="force_z_offset" value="0.115"/>

File: hexapod_description/urdf/modules/leg_hexaforce.xacro (robot description, xacro)
@@ -6,4 +6,13 @@
             <parent link="base_link"/>
             <child link="leg_${index}_1"/>
+            <xacro:if value="${(index+1) % 3 == 0}">
+                <xacro:property name="offset_limit" value= "0.57"/>
+            </xacro:if>
+            <xacro:if value="${(index+1) % 3 == 1}">
+                <xacro:property name="offset_limit" value= "-0.57"/>
+            </xacro:if>
+            <xacro:if value="${(index+1) % 3 == 2}">
+                <xacro:property name="offset_limit" value= "0"/>
+            </xacro:if>
             <limit effort="${joint_eff}" lower="${-joint_lim}" upper="${joint_lim}" velocity="${joint_vel}"/>
             <!-- Add a small offset angle to match the default position on the robot -->
@@ -57,5 +66,5 @@
             <parent link="leg_${index}_2"/>
             <child link="leg_${index}_3"/>
-            <limit effort="${joint_eff}" lower="${-joint_lim}" upper="${joint_lim}" velocity="${joint_vel}"/>
+            <limit effort="${joint_eff}" lower="${-joint_lim}" upper="0.82" velocity="${joint_vel}"/>
             <origin rpy="0 0 0" xyz="0.2 ${leg2_length+1} 0"/>
             <axis xyz="-1 0 0"/>

File: hexapod_description/urdf/modules/leg_pexod.xacro (robot description, xacro)
@@ -2,8 +2,17 @@
 <robot xmlns:xacro="http://www.ros.org/wiki/xacro">
   <!-- XACRO MACRO FOR LEGS LINKS/JOINTS -->
-    <xacro:macro name="leg" params="index xPos yPos">
+    <xacro:macro name="leg" params="index xPos yPos zPos">
         <joint name="body_leg_${index}" type="revolute">
             <parent link="base_link"/>
             <child link="leg_${index}_1"/>
+            <xacro:if value="${(index+1) % 3 == 0}">
+                <xacro:property name="offset_limit" value= "0.57"/>
+            </xacro:if>
+            <xacro:if value="${(index+1) % 3 == 1}">
+                <xacro:property name="offset_limit" value= "-0.57"/>
+            </xacro:if>
+            <xacro:if value="${(index+1) % 3 == 2}">
+                <xacro:property name="offset_limit" value= "0"/>
+            </xacro:if>
             <limit effort="${joint_eff}" lower="${-joint_lim}" upper="${joint_lim}" velocity="${joint_vel}"/>
             <!-- Add a small offset angle to match the default position on the robot -->
@@ -22,5 +31,5 @@
                 <xacro:property name="legs_rotation" value="${PI}"/>
             </xacro:if>
-            <origin rpy="0 0 ${offset_angle+legs_rotation}" xyz="${xPos} ${yPos} 0"/>
+            <origin rpy="0 0 ${offset_angle+legs_rotation}" xyz="${xPos} ${yPos} ${zPos}"/>
             <axis xyz="0 0 1"/>
             <dynamics damping="${joint_dmp}" friction="${joint_friction}"/>
@@ -40,5 +49,5 @@
             <child link="leg_${index}_2"/>
             <limit effort="${joint_eff}" lower="${-joint_lim}" upper="${joint_lim}" velocity="${joint_vel}"/>
-            <origin rpy="0 0 0" xyz="0 ${leg1_length} 0"/>
+            <origin rpy="0 0 0" xyz="-0.2 ${leg1_length+0.7} -0.2"/>
             <axis xyz="1 0 0"/>
             <dynamics damping="${joint_dmp}" friction="${joint_friction}"/>
@@ -57,6 +66,6 @@
             <parent link="leg_${index}_2"/>
             <child link="leg_${index}_3"/>
-            <limit effort="${joint_eff}" lower="${-joint_lim}" upper="${joint_lim}" velocity="${joint_vel}"/>
-            <origin rpy="0 0 0" xyz="0 ${leg2_length} 0"/>
+            <limit effort="${joint_eff}" lower="${-joint_lim}" upper="0.82" velocity="${joint_vel}"/>
+            <origin rpy="0 0 0" xyz="0.2 ${leg2_length+1} 0"/>
             <axis xyz="-1 0 0"/>
             <dynamics damping="${joint_dmp}" friction="${joint_friction}"/>

File: hexapod_description/urdf/modules/pexod.xacro (robot description, xacro)
@@ -6,5 +6,5 @@
   <xacro:property name="PI_4" value="0.78539816339" />
   <xacro:property name="scale" value="0.001" />
-  <xacro:property name="body_mass" value="1.031"/>
+  <xacro:property name="body_mass" value="1.834"/>
   <xacro:property name="body_length" value="0.24"/>
   <xacro:property name="body_width" value="0.119"/>
@@ -14,14 +14,14 @@
   <xacro:property name="leg1_length" value="0.06"/>
   <xacro:property name="leg1_dist" value="0.2"/>
-  <xacro:property name="leg1_mass" value="0.02"/>
+  <xacro:property name="leg1_mass" value="0.073"/>
   <xacro:property name="leg2_width" value="0.038"/>
   <xacro:property name="leg2_length" value="0.0835"/>
   <xacro:property name="leg2_dist" value="0.2"/>
-  <xacro:property name="leg2_mass" value="0.184"/>
+  <xacro:property name="leg2_mass" value="0.02"/>
   <xacro:property name="leg3_width" value="0.054"/>
   <xacro:property name="leg3_length" value="0.065"/>
   <xacro:property name="leg3_height" value="0.10"/>
   <xacro:property name="leg3_tip_radius" value="0.02"/>
-  <xacro:property name="leg3_mass" value="0.04"/>
+  <xacro:property name="leg3_mass" value="0.08"/>
   <xacro:property name="joint_lim" value="${PI_2}"/>
   <xacro:property name="joint_eff" value="2.5"/>

File: hexapod_description/urdf/pexod_visuals_collisions.xacro (robot description, xacro)
@@ -51,9 +51,9 @@
   <xacro:macro name="visuals_collisions_leg_1">
     <visual>
-      <origin xyz="0 0 0" rpy="0 ${PI_2} 0"/>
+      <origin xyz="0 0.75 0" rpy="-${PI} 0 0"/>
         <geometry>
           <mesh filename="${path_prefix + 'stl/first_link.stl'}" scale="0.001 0.001 0.001"/>
         </geometry>
-      <material name="Red"/>
+      <material name="Green"/>
     </visual>
     <collision>
@@ -66,5 +66,5 @@
   <xacro:macro name="visuals_collisions_leg_2">
     <visual>
-      <origin xyz="0 0 0" rpy="0 -${PI_2} 0"/>
+      <origin xyz="0 0 0" rpy="${PI_2} ${PI} ${PI_2}"/>
         <geometry>
           <mesh filename="${path_prefix + 'stl/second_link.stl'}" scale="0.001 0.001 0.001"/>
